Commit message: please work

File: src/mjbot_description/urdf/mjbot.urdf.xacro (robot description, xacro)
@@ -11,4 +11,3 @@
   <xacro:mjbot prefix="$(arg prefix)" />
   <xacro:mjbot_ros2_control   name="mjbot" />
-  <xacro:mjbot_arm_ros2_control name="mjbot" />
 </robot>

File: src/mjbot_description/urdf/ros2_control/mjbot_arm.ros2_control.xacro (robot description, xacro)
@@ -1,5 +1,5 @@
 <?xml version="1.0"?>
 <robot xmlns:xacro="http://www.ros.org/wiki/xacro">
-  <xacro:macro name="mjbot_arm_ros2_control" params="name">
+  <xacro:macro name="mjbot_ros2_control" params="name">
     <ros2_control name="${name}" type="system">
       <hardware>

File: src/mjbot_description/urdf/ros2_control/mjbot_base_control.urdf.xacro (robot description, xacro)
@@ -14,6 +14,10 @@
         <param name="enable_watchdog">0</param>
         <param name="watchdog_timeout">0.1</param>
-        <command_interface name="position"/>
-        <command_interface name="velocity"/>
+        <command_interface name="velocity">
+          <param name="min">-1</param>
+          <param name="max">1</param>
+        </command_interface>
+        <command_interface name="position" />
+        <command_interface name="effort" />
         <state_interface name="position"/>
         <state_interface name="velocity"/>
@@ -25,6 +29,10 @@
         <param name="enable_watchdog">0</param>
         <param name="watchdog_timeout">0.1</param>
-        <command_interface name="position"/>
-        <command_interface name="velocity"/>
+        <command_interface name="velocity">
+          <param name="min">-1</param>
+          <param name="max">1</param>
+        </command_interface>
+        <command_interface name="position" />
+        <command_interface name="effort" />
         <state_interface name="position"/>
         <state_interface name="velocity"/>

Commit message: arm mode

File: src/mjbot_description/urdf/mjbot.urdf.xacro (robot description, xacro)
@@ -11,3 +11,4 @@
   <xacro:mjbot prefix="$(arg prefix)" />
   <xacro:mjbot_ros2_control   name="mjbot" />
+  <xacro:mjbot_arm_ros2_control name="mjbot_arm" />
 </robot>

File: src/mjbot_description/urdf/ros2_control/mjbot_arm.ros2_control.xacro (robot description, xacro)
@@ -1,5 +1,5 @@
 <?xml version="1.0"?>
 <robot xmlns:xacro="http://www.ros.org/wiki/xacro">
-  <xacro:macro name="mjbot_ros2_control" params="name">
+  <xacro:macro name="mjbot_arm_ros2_control" params="name">
     <ros2_control name="${name}" type="system">
       <hardware>

File: src/mjbot_description/urdf/ros2_control/mjbot_base_control.urdf.xacro (robot description, xacro)
@@ -12,5 +12,5 @@
         <param name="serial_number">${serial_number}</param>
         <param name="axis">0</param>
-        <param name="enable_watchdog">0</param>
+        <param name="enable_watchdog">1</param>
         <param name="watchdog_timeout">0.1</param>
         <command_interface name="velocity">
@@ -27,5 +27,5 @@
         <param name="serial_number">${serial_number}</param>
         <param name="axis">1</param>
-        <param name="enable_watchdog">0</param>
+        <param name="enable_watchdog">1</param>
         <param name="watchdog_timeout">0.1</param>
         <command_interface name="velocity">

Commit message: commit

File: src/mjbot_description/urdf/mjbot.urdf.xacro (robot description, xacro)
@@ -8,7 +8,7 @@
   <!-- ros2_control -->
   <!-- <xacro:include filename="$(find mjbot_description)/urdf/ros2_control/mjbot_base_control.urdf.xacro" />
-  <xacro:include filename="$(find mjbot_description)/urdf/ros2_control/mjbot_arm.ros2_control.xacro" /> -->
+  <xacro:include filename="$(find mjbot_description)/urdf/ros2_control/mjbot_servos.ros2_control.xacro" /> -->
   <xacro:mjbot prefix="$(arg prefix)" />
-  <!-- <xacro:mjbot_ros2_control   name="mjbot_base" />
-  <xacro:mjbot_arm_ros2_control name="mjbot_arm" /> -->
+  <xacro:mjbot_ros2_control   name="mjbot_base" />
+  <xacro:mjbot_arm_ros2_control name="mjbot_servos" />
 </robot>

File: src/mjbot_description/urdf/ros2_control/mjbot_servos.ros2_control.xacro (robot description, xacro)
@@ -57,4 +57,12 @@
         <state_interface name="effort"/>
       </joint>
+      <joint name="neck">
+        <param name="id">3</param>
+        <command_interface name="position"/>
+        <command_interface name="velocity"/>
+        <state_interface name="position"/>
+        <state_interface name="velocity"/>
+        <state_interface name="effort"/>
+      </joint>
     </ros2_control>
   </xacro:macro>
