Commit message: comm

File: src/mjbot_description/urdf/ros2_control/mjbot_arm.ros2_control.xacro (robot description, xacro)
@@ -57,12 +57,4 @@
         <state_interface name="effort"/>
       </joint>
-      <joint name="neck">
-        <param name="id">3</param>
-        <command_interface name="position"/>
-        <command_interface name="velocity"/>
-        <state_interface name="position"/>
-        <state_interface name="velocity"/>
-        <state_interface name="effort"/>
-      </joint>
     </ros2_control>
   </xacro:macro>
